File: Projects/mech433.sch (EAGLE design)
At the start: 23 parts, among them J1 USB-MB-H

Commit message: Schematic update
Parts:
- added C7: .1uF, mech433:C-US025-025X050
Connections:
- net N$1 renamed VBUS
- new net A0: U$1.19.A0, U$8.1
- new net A1: U$1.20.A1, U$8.2
- new net A4: LED2.A, U$1.34.A4, U$8.6
- new net B13: U$9.3
- new net B14: U$1.14.B14, U$9.2
- new net B15: U$1.15.B15, U$9.1
- new net B2: U$1.23.B2, U$8.3
- new net B3: U$1.24.B3, U$8.4
- new net B4: U$1.33.B4, U$8.5
- new net B7: U$1.43.B7, U$9.6
- new net B8: U$1.B8, U$9.5
- new net B9: U$1.1.B9, U$1.11.B13, U$9.4
- new net D+: J1.D+, U$1.8.PGD2/B10
- new net D-: J1.D-, U$1.9.PGC2/B11
- new net MCLR: U$1.18.MCLR, U$7.1.MCLR
- new net N$6: C6.+, U$1.7.VCAP
- new net PGC1: U$1.22.B1, U$7.5.PGC
- new net PGD1: U$1.21.PGD1/B0, U$7.4.PGD
- new net USBID: J1.ID, U$1.41.B5
- net +3V3: now also C2.1, C7.1, U$1.10.VUSB3V3, U$1.17.AVDD, U$1.40.VDD, U$7.2.VDD, U$8.7; no longer LED2.A
- net +5V: now also U$9.7
- net GND: now also C6.-, C7.2, U$1.16.AVSS, U$1.6.VSS, U$7.3.GND, U$8.8, U$9.8
Other:
- moved on the sheet: C1, C2, C3, C4, C5, C6, J1, LED1, LED2, R1, R2, R3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

Commit message: Finished Schematic
Connections:
- net +3V3: now also R4.2, R5.2
- net B4: now also R5.1, U$6.1
- net GND: now also U$5.2, U$6.2
- net MCLR: now also R4.1, U$5.1
Other:
- moved on the sheet: R4, R5, U$5, U$6
Changed lines of the file:
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@@
 <part name="U$1" library="mech433" deviceset="PIC32MX250F256D" device=""/>
 <part name="P+1" library="mech433" deviceset="+5V" device=""/>
-<part name="P+2" library="mech433" deviceset="+5V" device=""/>
 <part name="J1" library="mech433" deviceset="USB" device="-MB-H"/>
 <part name="U$2" library="mech433" deviceset="SLIDE" device=""/>
@@
 <part name="GND23" library="mech433" deviceset="GND" device=""/>
 <part name="P+4" library="mech433" deviceset="+5V" device=""/>
+<part name="+3V8" library="mech433" deviceset="+3V3" device=""/>
+<part name="+3V9" library="mech433" deviceset="+3V3" device=""/>
 </parts>
 <sheets>
@@
 <attribute name="VALUE" x="40.64" y="88.9" size="1.778" layer="96" rot="R90"/>
 </instance>
-<instance part="P+2" gate="1" x="22.86" y="111.76" smashed="yes">
-<attribute name="VALUE" x="20.32" y="106.68" size="1.778" layer="96" rot="R90"/>
-</instance>
 <instance part="J1" gate="G$1" x="-15.24" y="81.28" smashed="yes" rot="MR0">
 <attribute name="NAME" x="-15.24" y="88.265" size="1.778" layer="95" rot="MR0"/>
@@
 <attribute name="VALUE" x="83.82" y="101.6" size="1.27" layer="94" rot="R180"/>
 </instance>
-<instance part="U$5" gate="G$1" x="162.56" y="86.36" smashed="yes">
-<attribute name="NAME" x="160.02" y="99.06" size="1.27" layer="94"/>
-<attribute name="VALUE" x="160.02" y="96.52" size="1.27" layer="94"/>
-</instance>
-<instance part="U$6" gate="G$1" x="162.56" y="66.04" smashed="yes">
-<attribute name="NAME" x="160.02" y="78.74" size="1.27" layer="94"/>
-<attribute name="VALUE" x="160.02" y="76.2" size="1.27" layer="94"/>
+<instance part="U$5" gate="G$1" x="121.92" y="-58.42" smashed="yes">
+<attribute name="NAME" x="119.38" y="-45.72" size="1.27" layer="94"/>
+<attribute name="VALUE" x="119.38" y="-48.26" size="1.27" layer="94"/>
+</instance>
+<instance part="U$6" gate="G$1" x="-7.62" y="-60.96" smashed="yes">
+<attribute name="NAME" x="-10.16" y="-48.26" size="1.27" layer="94"/>
+<attribute name="VALUE" x="-10.16" y="-50.8" size="1.27" layer="94"/>
 </instance>
 <instance part="U$7" gate="G$1" x="149.86" y="20.32" smashed="yes">
@@
 <attribute name="VALUE" x="127.762" y="74.93" size="1.778" layer="96" rot="R90"/>
 </instance>
-<instance part="R4" gate="G$1" x="144.78" y="99.06" smashed="yes">
-<attribute name="NAME" x="140.97" y="100.5586" size="1.778" layer="95"/>
-<attribute name="VALUE" x="140.97" y="95.758" size="1.778" layer="96"/>
+<instance part="R4" gate="G$1" x="106.68" y="-50.8" smashed="yes" rot="R90">
+<attribute name="NAME" x="105.1814" y="-54.61" size="1.778" layer="95" rot="R90"/>
+<attribute name="VALUE" x="109.982" y="-54.61" size="1.778" layer="96" rot="R90"/>
 </instance>
 <instance part="C1" gate="G$1" x="63.5" y="48.26" smashed="yes" rot="R90">
@@
 <attribute name="NAME" x="-43.18" y="-33.528" size="1.778" layer="95" font="vector" rot="MR180"/>
 </instance>
-<instance part="GND1" gate="1" x="-10.16" y="10.16" smashed="yes">
-<attribute name="VALUE" x="-12.7" y="7.62" size="1.778" layer="96"/>
+<instance part="GND1" gate="1" x="139.7" y="-63.5" smashed="yes">
+<attribute name="VALUE" x="137.16" y="-66.04" size="1.778" layer="96"/>
 </instance>
 <instance part="GND2" gate="1" x="114.3" y="-15.24" smashed="yes">
@@
 <attribute name="VALUE" x="76.2" y="116.84" size="1.778" layer="96" rot="R180"/>
 </instance>
-<instance part="GND7" gate="1" x="-7.62" y="104.14" smashed="yes" rot="R180">
-<attribute name="VALUE" x="-5.08" y="106.68" size="1.778" layer="96" rot="R180"/>
+<instance part="GND7" gate="1" x="12.7" y="-66.04" smashed="yes">
+<attribute name="VALUE" x="10.16" y="-68.58" size="1.778" layer="96"/>
 </instance>
 <instance part="GND8" gate="1" x="50.8" y="78.74" smashed="yes">
@@
 <attribute name="VALUE" x="101.6" y="78.74" size="1.778" layer="96"/>
 </instance>
-<instance part="R5" gate="G$1" x="139.7" y="58.42" smashed="yes">
-<attribute name="NAME" x="135.89" y="59.9186" size="1.778" layer="95"/>
-<attribute name="VALUE" x="135.89" y="55.118" size="1.778" layer="96"/>
+<instance part="R5" gate="G$1" x="-22.86" y="-53.34" smashed="yes" rot="R90">
+<attribute name="NAME" x="-24.3586" y="-57.15" size="1.778" layer="95" rot="R90"/>
+<attribute name="VALUE" x="-19.558" y="-57.15" size="1.778" layer="96" rot="R90"/>
 </instance>
 <instance part="GND17" gate="1" x="203.2" y="83.82" smashed="yes">
@@
 <instance part="P+4" gate="1" x="-25.4" y="-27.94" smashed="yes" rot="R270">
 <attribute name="VALUE" x="-22.86" y="-27.94" size="1.778" layer="96"/>
+</instance>
+<instance part="+3V8" gate="G$1" x="106.68" y="-38.1" smashed="yes">
+<attribute name="VALUE" x="104.14" y="-38.1" size="1.778" layer="96" rot="R90"/>
+</instance>
+<instance part="+3V9" gate="G$1" x="-22.86" y="-40.64" smashed="yes">
+<attribute name="VALUE" x="-15.24" y="-40.64" size="1.778" layer="96" rot="R180"/>
 </instance>
 </instances>
@@
 <wire x1="-33.02" y1="-30.48" x2="-27.94" y2="-30.48" width="0.1524" layer="91"/>
 <pinref part="GND23" gate="1" pin="GND"/>
+</segment>
+<segment>
+<pinref part="U$6" gate="G$1" pin="2"/>
+<wire x1="7.62" y1="-60.96" x2="12.7" y2="-60.96" width="0.1524" layer="91"/>
+<pinref part="GND7" gate="1" pin="GND"/>
+<wire x1="12.7" y1="-60.96" x2="12.7" y2="-63.5" width="0.1524" layer="91"/>
+</segment>
+<segment>
+<pinref part="U$5" gate="G$1" pin="2"/>
+<wire x1="137.16" y1="-58.42" x2="139.7" y2="-58.42" width="0.1524" layer="91"/>
+<pinref part="GND1" gate="1" pin="GND"/>
+<wire x1="139.7" y1="-58.42" x2="139.7" y2="-60.96" width="0.1524" layer="91"/>
 </segment>
 </net>
@@
 <pinref part="+3V7" gate="G$1" pin="+3V3"/>
 </segment>
+<segment>
+<pinref part="R4" gate="G$1" pin="2"/>
+<wire x1="106.68" y1="-45.72" x2="106.68" y2="-40.64" width="0.1524" layer="91"/>
+<pinref part="+3V8" gate="G$1" pin="+3V3"/>
+</segment>
+<segment>
+<pinref part="R5" gate="G$1" pin="2"/>
+<wire x1="-22.86" y1="-48.26" x2="-22.86" y2="-43.18" width="0.1524" layer="91"/>
+<pinref part="+3V9" gate="G$1" pin="+3V3"/>
+</segment>
 </net>
 <net name="N$5" class="0">
@@
 <label x="134.62" y="25.4" size="1.778" layer="95"/>
 </segment>
+<segment>
+<pinref part="U$5" gate="G$1" pin="1"/>
+<pinref part="R4" gate="G$1" pin="1"/>
+<wire x1="106.68" y1="-58.42" x2="106.68" y2="-55.88" width="0.1524" layer="91"/>
+<wire x1="106.68" y1="-58.42" x2="99.06" y2="-58.42" width="0.1524" layer="91"/>
+<junction x="106.68" y="-58.42"/>
+<label x="96.52" y="-58.42" size="1.778" layer="95"/>
+</segment>
 </net>
 <net name="A0" class="0">
@@
 <label x="134.62" y="-22.86" size="1.778" layer="95"/>
 </segment>
-</net>
+<segment>
+<pinref part="R5" gate="G$1" pin="1"/>
+<pinref part="U$6" gate="G$1" pin="1"/>
+<wire x1="-22.86" y1="-58.42" x2="-22.86" y2="-60.96" width="0.1524" layer="91"/>
+<wire x1="-22.86" y1="-60.96" x2="-33.02" y2="-60.96" width="0.1524" layer="91"/>
+<junction x="-22.86" y="-60.96"/>
+<label x="-30.48" y="-58.42" size="1.778" layer="95"/>
+</segment>
+</net>

Commit message: Making Board
Parts:
- removed R1: (no value), mech433:R-US_0207/10
Connections:
- net +3V3: now also U$4.3.VOUT; no longer U$4.2.VIN
- net +5V: now also U$4.2.VIN; no longer U$4.3.VOUT
- net B13: now also U$1.11.B13
- net B9: no longer U$1.11.B13
Other:
- moved on the sheet: U$4
Changed lines of the file:
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@@
 <?xml version="1.0" encoding="utf-8"?>
 <!DOCTYPE eagle SYSTEM "eagle.dtd">
-<eagle version="9.3.2">
+<eagle version="9.4.0">
 <drawing>
 <settings>
@@
 <part name="LED1" library="led" library_urn="urn:adsk.eagle:library:259" deviceset="LED" device="3MM" package3d_urn="urn:adsk.eagle:package:15797/1" value="Red"/>
 <part name="LED2" library="led" library_urn="urn:adsk.eagle:library:259" deviceset="LED" device="3MM" package3d_urn="urn:adsk.eagle:package:15797/1" value="Green"/>
-<part name="R1" library="mech433" deviceset="R-US_" device="0207/10" package3d_urn="urn:adsk.eagle:package:23491/2"/>
 <part name="R2" library="mech433" deviceset="R-US_" device="0207/10" package3d_urn="urn:adsk.eagle:package:23491/2" value="330"/>
 <part name="R3" library="mech433" deviceset="R-US_" device="0207/10" package3d_urn="urn:adsk.eagle:package:23491/2" value="330"/>
@@
 <part name="GND16" library="mech433" deviceset="GND" device=""/>
 <part name="R5" library="mech433" deviceset="R-US_" device="0207/10" package3d_urn="urn:adsk.eagle:package:23491/2" value="10K"/>
-<part name="GND17" library="mech433" deviceset="GND" device=""/>
-<part name="GND18" library="mech433" deviceset="GND" device=""/>
 <part name="C6" library="mech433" deviceset="CPOL-US" device="B45181B" package3d_urn="urn:adsk.eagle:package:23320/1" value="10uF"/>
 <part name="GND19" library="mech433" deviceset="GND" device=""/>
@@
 <attribute name="VALUE" x="53.34" y="53.34" size="1.27" layer="94" rot="MR90"/>
 </instance>
-<instance part="U$4" gate="G$1" x="73.66" y="93.98" smashed="yes" rot="R180">
-<attribute name="NAME" x="83.82" y="99.06" size="1.27" layer="94" rot="R180"/>
-<attribute name="VALUE" x="83.82" y="101.6" size="1.27" layer="94" rot="R180"/>
+<instance part="U$4" gate="G$1" x="73.66" y="93.98" smashed="yes">
+<attribute name="NAME" x="63.5" y="88.9" size="1.27" layer="94"/>
+<attribute name="VALUE" x="63.5" y="86.36" size="1.27" layer="94"/>
 </instance>
 <instance part="U$5" gate="G$1" x="121.92" y="-58.42" smashed="yes">
@@
 <attribute name="VALUE" x="130.175" y="86.868" size="1.778" layer="96" rot="R90"/>
 </instance>
-<instance part="R1" gate="G$1" x="104.14" y="109.22" smashed="yes">
-<attribute name="NAME" x="100.33" y="110.7186" size="1.778" layer="95"/>
-<attribute name="VALUE" x="100.33" y="105.918" size="1.778" layer="96"/>
-</instance>
 <instance part="R2" gate="G$1" x="114.3" y="78.74" smashed="yes" rot="R90">
 <attribute name="NAME" x="112.8014" y="74.93" size="1.778" layer="95" rot="R90"/>
@@
 <attribute name="VALUE" x="111.76" y="-17.78" size="1.778" layer="96"/>
 </instance>
-<instance part="GND3" gate="1" x="71.12" y="48.26" smashed="yes" rot="R90">
-<attribute name="VALUE" x="73.66" y="45.72" size="1.778" layer="96" rot="R90"/>
+<instance part="GND3" gate="1" x="73.66" y="48.26" smashed="yes" rot="R90">
+<attribute name="VALUE" x="76.2" y="45.72" size="1.778" layer="96" rot="R90"/>
 </instance>
 <instance part="GND4" gate="1" x="55.118" y="-43.18" smashed="yes">
@@
 <attribute name="VALUE" x="55.372" y="45.212" size="1.778" layer="96" rot="R180"/>
 </instance>
-<instance part="GND6" gate="1" x="73.66" y="114.3" smashed="yes" rot="R180">
-<attribute name="VALUE" x="76.2" y="116.84" size="1.778" layer="96" rot="R180"/>
+<instance part="GND6" gate="1" x="73.66" y="73.66" smashed="yes">
+<attribute name="VALUE" x="71.12" y="71.12" size="1.778" layer="96"/>
 </instance>
 <instance part="GND7" gate="1" x="12.7" y="-66.04" smashed="yes">
@@
 <attribute name="NAME" x="-24.3586" y="-57.15" size="1.778" layer="95" rot="R90"/>
 <attribute name="VALUE" x="-19.558" y="-57.15" size="1.778" layer="96" rot="R90"/>
-</instance>
-<instance part="GND17" gate="1" x="203.2" y="83.82" smashed="yes">
-<attribute name="VALUE" x="200.66" y="81.28" size="1.778" layer="96"/>
-</instance>
-<instance part="GND18" gate="1" x="203.2" y="101.6" smashed="yes">
-<attribute name="VALUE" x="200.66" y="99.06" size="1.778" layer="96"/>
 </instance>
 <instance part="C6" gate="G$1" x="63.5" y="-50.8" smashed="yes" rot="R90">
@@
 <pinref part="U$4" gate="G$1" pin="1.GND"/>
 <pinref part="GND6" gate="1" pin="GND"/>
-<wire x1="73.66" y1="109.22" x2="73.66" y2="111.76" width="0.1524" layer="91"/>
+<wire x1="73.66" y1="78.74" x2="73.66" y2="76.2" width="0.1524" layer="91"/>
 </segment>
 <segment>
@@
 <pinref part="GND3" gate="1" pin="GND"/>
 <pinref part="C1" gate="G$1" pin="2"/>
+<wire x1="71.12" y1="48.26" x2="68.58" y2="48.26" width="0.1524" layer="91"/>
 </segment>
 <segment>
@@
 <junction x="50.8" y="91.44"/>
 <wire x1="55.88" y1="91.44" x2="55.88" y2="93.98" width="0.1524" layer="91"/>
-<pinref part="U$4" gate="G$1" pin="3.VOUT"/>
+<pinref part="U$4" gate="G$1" pin="2.VIN"/>
 <wire x1="55.88" y1="93.98" x2="58.42" y2="93.98" width="0.1524" layer="91"/>
 </segment>
@@
 <net name="+3V3" class="0">
 <segment>
-<pinref part="U$4" gate="G$1" pin="2.VIN"/>
 <pinref part="C4" gate="G$1" pin="1"/>
-<wire x1="88.9" y1="93.98" x2="93.98" y2="93.98" width="0.1524" layer="91"/>
 <pinref part="C5" gate="G$1" pin="+"/>
 <wire x1="93.98" y1="93.98" x2="104.14" y2="93.98" width="0.1524" layer="91"/>
-<junction x="93.98" y="93.98"/>
 <pinref part="LED1" gate="G$1" pin="A"/>
 <wire x1="104.14" y1="93.98" x2="111.76" y2="93.98" width="0.1524" layer="91"/>
@@
 <pinref part="+3V2" gate="G$1" pin="+3V3"/>
 <junction x="111.76" y="93.98"/>
+<pinref part="U$4" gate="G$1" pin="3.VOUT"/>
+<wire x1="88.9" y1="93.98" x2="93.98" y2="93.98" width="0.1524" layer="91"/>
+<junction x="93.98" y="93.98"/>
 </segment>
 <segment>
@@
 <net name="B9" class="0">
 <segment>
-<pinref part="U$1" gate="G$1" pin="11.B13"/>
-<wire x1="80.733571875" y1="-37.90085" x2="80.733571875" y2="-45.72" width="0.1524" layer="91"/>
-<wire x1="80.733571875" y1="-45.72" x2="81.28" y2="-45.72" width="0.1524" layer="91"/>
-<label x="83.82" y="-40.64" size="1.778" layer="95"/>
-</segment>
-<segment>
 <pinref part="U$1" gate="G$1" pin="1.B9"/>
 <wire x1="29.933571875" y1="-37.90085" x2="29.933571875" y2="-45.72" width="0.1524" layer="91"/>
@@
 <label x="-25.4" y="-17.78" size="1.778" layer="95"/>
 </segment>
-</net>
+<segment>
+<pinref part="U$1" gate="G$1" pin="11.B13"/>
+<wire x1="80.733571875" y1="-37.90085" x2="80.733571875" y2="-45.72" width="0.1524" layer="91"/>
+<wire x1="80.733571875" y1="-45.72" x2="81.28" y2="-45.72" width="0.1524" layer="91"/>
+<label x="83.82" y="-40.64" size="1.778" layer="95"/>
+</segment>
+</net>
